Commit message: update gazebo param

File: iiwa7_description/gazebo/iiwa.gazebo.xacro (robot description, xacro)
@@ -15,7 +15,7 @@
     </gazebo>
     <!-- color -->
-    <gazebo reference="${prefix}link_7">
+    <!-- <gazebo reference="${prefix}_link_7">
       <material>Gazebo/Gray</material>
-    </gazebo>
+    </gazebo> -->
   </xacro:macro>
 </robot>

File: iiwa7_description/urdf/iiwa7.urdf.xacro (robot description, xacro)
@@ -285,5 +285,5 @@
             <dynamics damping="${joint_damping}"/>
         </joint>
-        <joint name="${prefix}joint_6" type="revolute">
+        <joint name="${prefix}_joint_6" type="revolute">
             <origin xyz="0 0.06070 0.19" rpy="${PI / 2} 0 0"/>
             <parent link="${prefix}_link_5"/>

Commit message: old environment

File: iiwa7_description/gazebo/iiwa.gazebo.xacro (robot description, xacro)
@@ -15,7 +15,51 @@
     </gazebo>
     <!-- color -->
-    <!-- <gazebo reference="${prefix}_link_7">
-      <material>Gazebo/Gray</material>
-    </gazebo> -->
+    <gazebo reference="${prefix}_link_0">
+      <material>Gazebo/Grey</material>
+      <mu1>0.2</mu1>
+      <mu2>0.2</mu2>
+    </gazebo>
+    <!-- Link1 -->
+    <gazebo reference="${prefix}_link_1">
+      <material>Gazebo/Orange</material>
+      <mu1>0.2</mu1>
+      <mu2>0.2</mu2>
+    </gazebo>
+    <!-- Link2 -->
+    <gazebo reference="${prefix}_link_2">
+      <material>Gazebo/Orange</material>
+      <mu1>0.2</mu1>
+      <mu2>0.2</mu2>
+    </gazebo>
+    <!-- Link3 -->
+    <gazebo reference="${prefix}_link_3">
+      <material>Gazebo/Orange</material>
+      <mu1>0.2</mu1>
+      <mu2>0.2</mu2>
+    </gazebo>
+    <!-- Link4 -->
+    <gazebo reference="${prefix}_link_4">
+      <material>Gazebo/Orange</material>
+      <mu1>0.2</mu1>
+      <mu2>0.2</mu2>
+    </gazebo>
+    <!-- Link5 -->
+    <gazebo reference="${prefix}_link_5">
+      <material>Gazebo/Orange</material>
+      <mu1>0.2</mu1>
+      <mu2>0.2</mu2>
+    </gazebo>
+    <!-- Link6 -->
+    <gazebo reference="${prefix}_link_6">
+      <material>Gazebo/Orange</material>
+      <mu1>0.2</mu1>
+      <mu2>0.2</mu2>
+    </gazebo>
+    <!-- Link7 -->
+    <gazebo reference="${prefix}_link_7">
+      <material>Gazebo/Grey</material>
+      <mu1>0.2</mu1>
+      <mu2>0.2</mu2>
+    </gazebo>
   </xacro:macro>
 </robot>

File: iiwa7_description/urdf/iiwa7.urdf (robot description, URDF)
Before this commit: robot iiwa, 10 links, 9 joints
Links:
- link iiwa7_link_0: geometry collision mesh filename=package://iiwa_description/meshes/lbr_iiwa_14_r820/collisio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; visual mesh filename=package://iiwa_description/meshes/lbr_iiwa_14_r820/visual/b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
- link iiwa7_link_1: geometry collision mesh filename=package://iiwa_description/meshes/lbr_iiwa_14_r820/collisio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; visual mesh filename=package://iiwa_description/meshes/lbr_iiwa_14_r820/visual/l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
- link iiwa7_link_2: geometry collision mesh filename=package://iiwa_description/meshes/lbr_iiwa_14_r820/collisio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; visual mesh filename=package://iiwa_description/meshes/lbr_iiwa_14_r820/visual/l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
- link iiwa7_link_3: geometry collision mesh filename=package://iiwa_description/meshes/lbr_iiwa_14_r820/collisio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; visual mesh filename=package://iiwa_description/meshes/lbr_iiwa_14_r820/visual/l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
- link iiwa7_link_4: geometry collision mesh filename=package://iiwa_description/meshes/lbr_iiwa_14_r820/collisio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; visual mesh filename=package://iiwa_description/meshes/lbr_iiwa_14_r820/visual/l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
- link iiwa7_link_5: geometry collision mesh filename=package://iiwa_description/meshes/lbr_iiwa_14_r820/collisio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; visual mesh filename=package://iiwa_description/meshes/lbr_iiwa_14_r820/visual/l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
- link iiwa7_link_6: geometry collision mesh filename=package://iiwa_description/meshes/lbr_iiwa_14_r820/collisio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; visual mesh filename=package://iiwa_description/meshes/lbr_iiwa_14_r820/visual/l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
- link iiwa7_link_7: geometry collision mesh filename=package://iiwa_description/meshes/lbr_iiwa_14_r820/collisio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; visual mesh filename=package://iiwa_description/meshes/lbr_iiwa_14_r820/visual/l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
Joints:
- removed joint iiwa7joint_6
- removed joint iiwa7joint_a7-tool0
- added joint iiwa7_joint_6: type revolute, parent iiwa7_link_5, child iiwa7_link_6, origin xyz=0 0.06070 0.19 rpy=1.5707963267948966 0 0, axis 0 0 1, limit lower=-2.0943951023931953 upper=2.0943951023931953 effort=40 velocity=3.141592653589793
- added joint iiwa7_joint_7-tool0: type fixed, parent iiwa7_link_7, child iiwa7_tool0, origin xyz=0 0 0.045 rpy=0 0 0, axis 0 0 0

File: iiwa7_description/urdf/iiwa7.urdf.xacro (robot description, xacro)
@@ -199,5 +199,5 @@
                 <material name="gray"/>
                 <geometry>
-                    <mesh filename="package://iiwa7_description/meshes/iiwa7/visual/link_7_2.stl" />
+                    <mesh filename="package://iiwa7_description/meshes/iiwa7/visual/link_7.stl" />
                 </geometry>
             </visual>
@@ -205,5 +205,5 @@
                 <origin rpy="0 0 0" xyz="0 0 -0.0005"/>
                 <geometry>
-                <mesh filename="package://iiwa7_description/meshes/iiwa7/collision/link_7_2.stl" />
+                <mesh filename="package://iiwa7_description/meshes/iiwa7/collision/link_7.stl" />
                 </geometry>
             </collision>

File: iiwa7_description/urdf/iiwa7.xacro (robot description, xacro)
@@ -23,4 +23,8 @@
     <!-- Import all Gazebo-customization elements -->
     <xacro:include filename="$(find ${description_package})/gazebo/iiwa.gazebo.xacro"/>
+    <!-- Import Robot Base Station -->
+    <xacro:include filename="$(find ${description_package})/urdf/environment/base_table.xacro"/>
+    <!-- Import Conveyor Belt System -->
+    <xacro:include filename="$(find ${description_package})/urdf/environment/conveyor.xacro"/>
     <!-- Used for fixing robot -->
     <link name="world"/>
@@ -28,5 +32,13 @@
         <static>true</static>
     </gazebo>
-    <xacro:iiwa7 parent="world" prefix="$(arg prefix)">
+    <!-- World to table -->
+    <xacro:add_table table_link="$(arg prefix)_table_base" parent="world">
+        <origin xyz="0 0 1" rpy="0 0 0" />
+    </xacro:add_table>
+    <!-- World to Conveyor Belt -->
+    <xacro:conveyor_system parent="world">
+        <origin xyz="-1 -5.5 1" rpy="0 0 1.57" />
+    </xacro:conveyor_system>
+    <xacro:iiwa7 parent="$(arg prefix)_table_base" prefix="$(arg prefix)">
         <origin xyz="0 0 0" rpy="0 0 0" />
     </xacro:iiwa7>
