Commit message: added extra collision

File: iiwa7_description/urdf/environment/hochregallager.xacro (robot description, xacro)
@@ -64,4 +64,31 @@
         <origin xyz="0.05 -0.55 1.335" rpy="0 0 1.5708"/>
     </joint>
+    <link name="cable_box">
+      <inertial>
+        <mass value="100"/>
+        <origin xyz="0 0 0" />
+        <inertia  ixx="1" ixy="0.0"  ixz="0.0"  iyy="1"  iyz="0.0"  izz="1" />
+      </inertial>
+      <!-- <visual>
+        <origin rpy="0 0 0" xyz="0 0 0"/>
+        <geometry>
+          <box size="0.08 0.08 0.4"/>
+        </geometry>
+        <material name="white">
+          <color rgba="1.0 1.0 1.0 1.0"/>
+        </material>
+      </visual> -->
+      <collision>
+        <origin rpy="0 0 0" xyz="0 0 0"/>
+          <geometry>
+            <box size="0.08 0.08 0.4"/>
+          </geometry>
+      </collision>
+    </link>
+    <joint name="world_cable_box_joint" type="fixed">
+        <parent link="${parent}"/>
+        <child link="cable_box"/>
+        <origin xyz="0.35 0.47 1.35" rpy="0 0 0"/>
+    </joint>
   </xacro:macro>
 </robot>
