Commit message: attach grippers

File: iiwa7_description/urdf/iiwa7.xacro (robot description, xacro)
@@ -29,4 +29,6 @@
     <!-- Import Hochregallager -->
     <xacro:include filename="$(find ${description_package})/urdf/environment/hochregallager.xacro"/>
+    <!-- Import Schunk WSG50 Gripper -->
+    <xacro:include filename="$(find wsg50_description)/urdf/wsg50.urdf.xacro"/>
     <!-- Used for fixing robot -->
     <link name="world"/>
@@ -63,3 +65,6 @@
         prefix="$(arg prefix)"
         />
+     <xacro:wsg50 prefix="wsg50" parent="$(arg prefix)_tool0" finger_length="0.023" finger_tip="-0.001">
+        <origin xyz="0 0 0" rpy="0 0 0" />
+    </xacro:wsg50>
 </robot>

Commit message: improve collision factors

File: iiwa7_description/urdf/iiwa7.xacro (robot description, xacro)
@@ -66,5 +66,5 @@
         />
      <xacro:wsg50 prefix="wsg50" parent="$(arg prefix)_tool0" finger_length="0.023" finger_tip="-0.001">
-        <origin xyz="0 0 0" rpy="0 0 0" />
+        <origin xyz="0 0 0.037" rpy="0 0 0" />
     </xacro:wsg50>
 </robot>

Commit message: change robot IP and update gripper orientation

File: iiwa7_description/urdf/iiwa7.xacro (robot description, xacro)
@@ -66,5 +66,5 @@
         />
      <xacro:wsg50 prefix="wsg50" parent="$(arg prefix)_tool0" finger_length="0.023" finger_tip="-0.001">
-        <origin xyz="0 0 0.037" rpy="0 0 0" />
+        <origin xyz="0 0 0.037" rpy="0 0 0.785398" />
     </xacro:wsg50>
 </robot>
