Commit message: todo: More test require to define the proper robot position

File: iiwa7_description/urdf/iiwa7.urdf.xacro (robot description, xacro)
@@ -3,4 +3,5 @@
     <!-- some parameters -->
     <xacro:property name="safety" value="true"/>
+    <xacro:property name="PI" value="3.1415926535897931"/>
     <!-- some constants -->
     <xacro:property name="safety_controller_k_pos" value="100"/>
