Commit message: TOdo

File: iiwa7_description/urdf/iiwa7.urdf (robot description, URDF)
Before this commit: robot iiwa, 10 links, 9 joints
Links:
- removed link iiwa7_link_0
- removed link iiwa7_link_1
- removed link iiwa7_link_2
- removed link iiwa7_link_3
- removed link iiwa7_link_4
- removed link iiwa7_link_5
- removed link iiwa7_link_6
- removed link iiwa7_link_7
- removed link iiwa7_tool0
- removed link world
Joints:
- removed joint iiwa7_base_joint
- removed joint iiwa7_joint_1
- removed joint iiwa7_joint_2
- removed joint iiwa7_joint_3
- removed joint iiwa7_joint_4
- removed joint iiwa7_joint_5
- removed joint iiwa7_joint_7
- removed joint iiwa7joint_6
- removed joint iiwa7joint_a7-tool0

Commit message: Complete env launch

File: iiwa7_description/urdf/iiwa7.urdf (robot description, URDF)
Before this commit: robot iiwa, 10 links, 9 joints
Links:
- added link conveyor_system_link, mass 100; collision mesh filename=package://iiwa7_description/meshes/conveyor/collision/bandu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 scale=0.001 0.001 0.001; visual mesh filename=package://iiwa7_description/meshes/conveyor/visual/bandumla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 scale=0.001 0.001 0.001
- added link display, mass 100; collision box size=0.55 0.01 0.67; visual box size=0.55 0.01 0.67
- added link iiwa7_table_base, mass 80; collision mesh filename=package://iiwa7_description/meshes/lf044_rough.stl scale=0.001 0.001 0.001; visual mesh filename=package://iiwa7_description/meshes/lf044_rough.dae scale=0.001 0.001 0.001
- added link table_ee, mass 1; collision box size=0.2 0.2 0.2; visual box size=0.2 0.2 0.03
- link iiwa7_link_0: geometry collision mesh filename=package://iiwa7_description/meshes/iiwa7/collision/link_0.s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; visual mesh filename=package://iiwa7_description/meshes/iiwa7/visual/link_0.dae
- link iiwa7_link_1: geometry collision mesh filename=package://iiwa7_description/meshes/iiwa7/collision/link_1.s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; visual mesh filename=package://iiwa7_description/meshes/iiwa7/visual/link_1.dae
- link iiwa7_link_2: geometry collision mesh filename=package://iiwa7_description/meshes/iiwa7/collision/link_2.s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; visual mesh filename=package://iiwa7_description/meshes/iiwa7/visual/link_2.dae
- link iiwa7_link_3: geometry collision mesh filename=package://iiwa7_description/meshes/iiwa7/collision/link_3.s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; visual mesh filename=package://iiwa7_description/meshes/iiwa7/visual/link_3.dae
- link iiwa7_link_4: geometry collision mesh filename=package://iiwa7_description/meshes/iiwa7/collision/link_4.s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; visual mesh filename=package://iiwa7_description/meshes/iiwa7/visual/link_4.dae
- link iiwa7_link_5: geometry collision mesh filename=package://iiwa7_description/meshes/iiwa7/collision/link_5.s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; visual mesh filename=package://iiwa7_description/meshes/iiwa7/visual/link_5.dae
- link iiwa7_link_6: geometry collision mesh filename=package://iiwa7_description/meshes/iiwa7/collision/link_6.s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; visual mesh filename=package://iiwa7_description/meshes/iiwa7/visual/link_6.dae
- link iiwa7_link_7: geometry collision mesh filename=package://iiwa7_description/meshes/iiwa7/collision/link_7.s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; visual mesh filename=package://iiwa7_description/meshes/iiwa7/visual/link_7.stl
Joints:
- added joint table_ee_joint: type fixed, parent iiwa7_table_base, child table_ee, origin xyz=0 0 -0.015 rpy=0 0 0
- added joint world_conveyor_joint: type fixed, parent world, child conveyor_system_link, origin xyz=-1 -5.5 1 rpy=0 0 1.57
- added joint world_display_joint: type fixed, parent world, child display, origin xyz=0 -0.6 1.335
- added joint world_iiwa7_table_base_table_joint: type fixed, parent world, child iiwa7_table_base, origin xyz=0 0 1 rpy=0 0 0
- joint iiwa7_base_joint: parent world -> iiwa7_table_base

Commit message: Complete environment

File: iiwa7_description/urdf/iiwa7.urdf (robot description, URDF)
Before this commit: robot iiwa, 14 links, 13 joints
Links:
- added link display_regal, mass 100; collision box size=0.55 0.01 0.67; visual box size=0.55 0.01 0.67
- added link hochregallager_link, mass 100; collision mesh filename=package://iiwa7_description/meshes/hochregallager/collision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 scale=0.001 0.001 0.001; visual mesh filename=package://iiwa7_description/meshes/hochregallager/visual/Ho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 scale=0.001 0.001 0.001
Joints:
- added joint world_hochregallager_joint: type fixed, parent world, child hochregallager_link, origin xyz=-1 -5.5 1 rpy=0 0 1.57
- joint world_display_joint: child display -> display_regal; parent world -> hochregallager_link

File: iiwa7_description/urdf/iiwa7.xacro (robot description, xacro)
@@ -27,4 +27,6 @@
     <!-- Import Conveyor Belt System -->
     <xacro:include filename="$(find ${description_package})/urdf/environment/conveyor.xacro"/>
+    <!-- Import Hochregallager -->
+    <xacro:include filename="$(find ${description_package})/urdf/environment/hochregallager.xacro"/>
     <!-- Used for fixing robot -->
     <link name="world"/>
@@ -40,4 +42,9 @@
         <origin xyz="-1 -5.5 1" rpy="0 0 1.57" />
     </xacro:conveyor_system>
+    <!-- World to Hochregallager -->
+    <xacro:hochregallager_system parent="world">
+        <origin xyz="0.80 -0.165 0" rpy="0 0 3.14159" />
+    </xacro:hochregallager_system>
+    <!-- table to iiwa7 -->
     <xacro:iiwa7 parent="$(arg prefix)_table_base" prefix="$(arg prefix)">
         <origin xyz="0 0 0" rpy="0 0 0" />

Commit message: isaac sim init

File: iiwa7_description/urdf/iiwa7.urdf (robot description, URDF)
Before this commit: robot iiwa, 16 links, 14 joints
Links:
- added link cable_box, mass 100; collision box size=0.08 0.08 0.4
- added link wsg50_base_link, mass 0.25; collision box size=0.25 0.09 0.0735; visual box size=0.20 0.09 0.0735
- added link wsg50_center
- added link wsg50_gripper_left, mass 0.1; collision mesh filename=package://wsg50_description/meshes/kuka_gripper_2.stl; visual mesh filename=package://wsg50_description/meshes/kuka_gripper_2.dae
- added link wsg50_gripper_right, mass 0.1; collision mesh filename=package://wsg50_description/meshes/kuka_gripper_2.stl; visual mesh filename=package://wsg50_description/meshes/kuka_gripper_2.dae
- link display_regal: geometry collision box size=0.65 0.01 0.75; visual box size=0.65 0.01 0.75
- link hochregallager_link: geometry collision mesh filename=package://iiwa7_description/meshes/hochregallager/collision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; visual mesh filename=package://iiwa7_description/meshes/hochregallager/visual/Ho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
Joints:
- added joint hochregallager_display_joint: type fixed, parent hochregallager_link, child display_regal, origin xyz=0.05 -0.55 1.335 rpy=0 0 1.5708
- added joint world_cable_box_joint: type fixed, parent world, child cable_box, origin xyz=0.35 0.47 1.35 rpy=0 0 0
- added joint wsg50_center_joint: type fixed, parent wsg50_base_link, child wsg50_center, origin xyz=0 0 0.023 rpy=0 0 0
- added joint wsg50_finger_left_joint: type fixed, parent wsg50_base_link, child wsg50_gripper_left, origin xyz=0.08 0 0.12 rpy=3.1457 0 3.1457, axis 1 0 0, limit lower=-0.055 upper=-0.0027 effort=1.0 velocity=1.0
- added joint wsg50_finger_right_joint: type fixed, parent wsg50_base_link, child wsg50_gripper_right, origin xyz=-0.08 0 0.12 rpy=3.14159 0 0, axis -1 0 0, limit lower=0.0027 upper=0.055 effort=1.0 velocity=1.0
- added joint wsg50_gripper_joint: type fixed, parent iiwa7_tool0, child wsg50_base_link, origin xyz=0 0 0.037 rpy=0 0 0.785398
- joint world_display_joint: child display_regal -> display; parent hochregallager_link -> world
- joint world_hochregallager_joint: origin xyz=-1 -5.5 1 rpy=0 0 1.57 -> xyz=0.80 -0.165 0 rpy=0 0 3.14159
