Commit message: Auto stash before merge of "main" and "origin/main"

File: iiwa7_description/ros2_control/iiwa.r2c_hardware.xacro (robot description, xacro)
@@ -101,5 +101,5 @@
                 <state_interface name="effort"/>
             </joint>
-            <sensor name="${prefix}external_torque_sensor">
+            <sensor name="external_torque_sensor">
                 <state_interface name="external_torque.joint_1"/>
                 <state_interface name="external_torque.joint_2"/>

File: iiwa7_description/urdf/iiwa7.urdf (robot description, URDF)
Before this commit: robot None, 0 links, 0 joints
Links:
- added link iiwa7_link_0, mass 5; collision mesh filename=package://iiwa7_description/meshes/iiwa7/collision/link_0.s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; visual mesh filename=package://iiwa7_description/meshes/iiwa7/visual/link_0.dae
- added link iiwa7_link_1, mass 3.4525; collision mesh filename=package://iiwa7_description/meshes/iiwa7/collision/link_1.s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; visual mesh filename=package://iiwa7_description/meshes/iiwa7/visual/link_1.dae
- added link iiwa7_link_2, mass 3.4821; collision mesh filename=package://iiwa7_description/meshes/iiwa7/collision/link_2.s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; visual mesh filename=package://iiwa7_description/meshes/iiwa7/visual/link_2.dae
- added link iiwa7_link_3, mass 4.05623; collision mesh filename=package://iiwa7_description/meshes/iiwa7/collision/link_3.s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; visual mesh filename=package://iiwa7_description/meshes/iiwa7/visual/link_3.dae
- added link iiwa7_link_4, mass 3.4822; collision mesh filename=package://iiwa7_description/meshes/iiwa7/collision/link_4.s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; visual mesh filename=package://iiwa7_description/meshes/iiwa7/visual/link_4.dae
- added link iiwa7_link_5, mass 2.1633; collision mesh filename=package://iiwa7_description/meshes/iiwa7/collision/link_5.s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; visual mesh filename=package://iiwa7_description/meshes/iiwa7/visual/link_5.dae
- added link iiwa7_link_6, mass 2.3466; collision mesh filename=package://iiwa7_description/meshes/iiwa7/collision/link_6.s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; visual mesh filename=package://iiwa7_description/meshes/iiwa7/visual/link_6.dae
- added link iiwa7_link_7, mass 3.129; collision mesh filename=package://iiwa7_description/meshes/iiwa7/collision/link_7_2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; visual mesh filename=package://iiwa7_description/meshes/iiwa7/visual/link_7_2.stl
- added link iiwa7_tool0
- added link world
Joints:
- added joint iiwa7_base_joint: type fixed, parent world, child iiwa7_link_0, origin xyz=0 0 0 rpy=0 0 0
- added joint iiwa7_joint_1: type revolute, parent iiwa7_link_0, child iiwa7_link_1, origin xyz=0 0 0.15 rpy=0 0 0, axis 0 0 1, limit lower=-2.9670597283903604 upper=2.9670597283903604 effort=176 velocity=1.710422666954443
- added joint iiwa7_joint_2: type revolute, parent iiwa7_link_1, child iiwa7_link_2, origin xyz=0 0 0.19 rpy=1.5707963267948966   0 3.141592653589793, axis 0 0 1, limit lower=-2.0943951023931953 upper=2.0943951023931953 effort=176 velocity=1.710422666954443
- added joint iiwa7_joint_3: type revolute, parent iiwa7_link_2, child iiwa7_link_3, origin xyz=0 0.21 0 rpy=1.5707963267948966 0 3.141592653589793, axis 0 0 1, limit lower=-2.9670597283903604 upper=2.9670597283903604 effort=110 velocity=1.7453292519943295
- added joint iiwa7_joint_4: type revolute, parent iiwa7_link_3, child iiwa7_link_4, origin xyz=0 0 0.19 rpy=1.5707963267948966 0 0, axis 0 0 1, limit lower=-2.0943951023931953 upper=2.0943951023931953 effort=110 velocity=2.2689280275926285
- added joint iiwa7_joint_5: type revolute, parent iiwa7_link_4, child iiwa7_link_5, origin xyz=0 0.21 0 rpy=-1.5707963267948966 3.141592653589793 0, axis 0 0 1, limit lower=-2.9670597283903604 upper=2.9670597283903604 effort=110 velocity=2.443460952792061
- added joint iiwa7_joint_7: type revolute, parent iiwa7_link_6, child iiwa7_link_7, origin xyz=0 0.081 0.06070 rpy=-1.5707963267948966 3.141592653589793 0, axis 0 0 1, limit lower=-3.0543261909900763 upper=3.0543261909900763 effort=40 velocity=3.141592653589793
- added joint iiwa7joint_6: type revolute, parent iiwa7_link_5, child iiwa7_link_6, origin xyz=0 0.06070 0.19 rpy=1.5707963267948966 0 0, axis 0 0 1, limit lower=-2.0943951023931953 upper=2.0943951023931953 effort=40 velocity=3.141592653589793
- added joint iiwa7joint_a7-tool0: type fixed, parent iiwa7link_7, child iiwa7tool0, origin xyz=0 0 0.045 rpy=0 0 0, axis 0 0 0

File: iiwa7_description/urdf/iiwa7.urdf.xacro (robot description, xacro)
@@ -61,5 +61,4 @@
                     <mesh filename="package://iiwa7_description/meshes/iiwa7/visual/link_0.dae"/>
                 </geometry>
-                <material name="Grey"/>
             </visual>
             <collision>
@@ -68,5 +67,4 @@
                     <mesh filename="package://iiwa7_description/meshes/iiwa7/collision/link_0.stl"/>
                 </geometry>
-                <material name="Grey"/>
             </collision>
             <inertial>
@@ -315,8 +313,8 @@
             <dynamics damping="${joint_damping}"/>
         </joint>
-        <joint name="${prefix}joint_a7-tool0" type="fixed">
+        <joint name="${prefix}_joint_7-tool0" type="fixed">
             <origin xyz="0 0 0.045" rpy="0 0 0"/>
-            <parent link="${prefix}link_7"/>
-            <child link="${prefix}tool0"/>
+            <parent link="${prefix}_link_7"/>
+            <child link="${prefix}_tool0"/>
             <axis xyz="0 0 0"/>
         </joint>

File: iiwa7_description/urdf/iiwa7.xacro (robot description, xacro)
@@ -10,4 +10,5 @@
     <xacro:arg name="command_interface" default="position" />
     <xacro:arg name="base_frame_file" default="base_frame.yaml" />
+    <xacro:arg name="initial_positions_file" default="initial_positions.yaml" />
     <xacro:arg name="description_package" default="iiwa7_description" />
     <xacro:arg name="runtime_config_package" default="iiwa7_description" />
@@ -15,5 +16,4 @@
     <xacro:arg name="namespace" default="/" />
     <xacro:property name="description_package" value="$(arg description_package)"/>
-    <xacro:arg name="initial_positions_file" default="$(find ${description_package})/config/initial_positions.yaml" />
     <xacro:property name="PI" value="3.1415926535897931"/>
     <!-- Import iiwa urdf file -->
@@ -35,5 +35,5 @@
         robot_ip="$(arg robot_ip)" robot_port="$(arg robot_port)"
         command_interface="$(arg command_interface)"
-        initial_positions_file="$(arg initial_positions_file)"
+        initial_positions_file="$(find ${description_package})/config/$(arg initial_positions_file)"
         use_sim="$(arg use_sim)" use_fake_hardware="$(arg use_fake_hardware)"
         />

Commit message: update loading xacro param

File: iiwa7_description/ros2_control/iiwa.r2c_hardware.xacro (robot description, xacro)
@@ -2,5 +2,5 @@
 <robot xmlns:xacro="http://www.ros.org/wiki/xacro">
     <xacro:macro name="iiwa_r2c_hardware" params="name prefix command_interface robot_ip robot_port initial_positions_file use_sim:=^|false use_fake_hardware:=^|true">
-        <xacro:property name="initial_positions" value="${load_yaml(initial_positions_file)['initial_positions']}"/>
+        <xacro:property name="initial_positions" value="${xacro.load_yaml(initial_positions_file)['initial_positions']}"/>
         <ros2_control name="${name}" type="system">
             <xacro:if value="$(arg use_sim)">
